Commit message: run test gazebo

File: catkin_ws/src/vis_lecture/xacro/body.xacro (robot description, xacro)
@@ -4,13 +4,16 @@
   <xacro:property name="body_width" value="0.4" />
   <xacro:property name="body_height" value="0.4" />
+  <xacro:property name="tire_height" value="0.1" />
   <xacro:include filename="tire.xacro" />
   <material name="green">
     <color rgba="${gcolor}" />
   </material>
-  <link name="base_link" />
+  <link name="base_link">
+    <origin xyz="0 0 ${tire_height}" rpy="0 0 0" />
+  </link>
   <joint name="body_joint" type="fixed">
     <parent link="base_link"/>
     <child  link="body_link"/>
-    <origin xyz="0 0 0" rpy="0 0 0" />
+    <origin xyz="0 0 ${tire_height}" rpy="0 0 0" />
   </joint>
   <link name="body_link">
@@ -23,7 +26,7 @@
     </visual>
   </link>
-  <xacro:make_tire suffix="tire0" parent="body_link" xyz="${body_width/2} ${body_height/2+tire_width/2} 0.0" rpy="0 1.57 -1.57" radius="0.1" length="${tire_width}"/>
-  <xacro:make_tire suffix="tire1" parent="body_link" xyz="${-(body_width/2)} ${body_height/2+tire_width/2} 0.0" rpy="0 1.57 -1.57" radius="0.1" length="${tire_width}"/>
-  <xacro:make_tire suffix="tire2" parent="body_link" xyz="${body_width/2} ${-(body_height/2+tire_width/2)} 0.0" rpy="0 1.57 1.57" radius="0.1" length="${tire_width}"/>
-  <xacro:make_tire suffix="tire3" parent="body_link" xyz="${-(body_width/2)} ${-(body_height/2+tire_width/2)} 0.0" rpy="0 1.57 1.57" radius="0.1" length="${tire_width}"/>
+  <xacro:make_tire suffix="tire0" parent="body_link" xyz="${body_width/2} ${body_height/2+tire_width/2} 0" rpy="0 1.57 -1.57" radius="${tire_height}" length="${tire_width}"/>
+  <xacro:make_tire suffix="tire1" parent="body_link" xyz="${-(body_width/2)} ${body_height/2+tire_width/2} 0" rpy="0 1.57 -1.57" radius="${tire_height}" length="${tire_width}"/>
+  <xacro:make_tire suffix="tire2" parent="body_link" xyz="${body_width/2} ${-(body_height/2+tire_width/2)} 0" rpy="0 1.57 1.57" radius="${tire_height}" length="${tire_width}"/>
+  <xacro:make_tire suffix="tire3" parent="body_link" xyz="${-(body_width/2)} ${-(body_height/2+tire_width/2)} 0" rpy="0 1.57 1.57" radius="${tire_height}" length="${tire_width}"/>
 </robot>

File: catkin_ws/src/vis_lecture/xacro/simple_car.xacro (robot description, xacro)
@@ -16,4 +16,9 @@
     </joint>
     <link name="${prefix}_link">
+      <inertial>
+        <origin xyz="0 0 0" rpy="0 0 0" />
+        <mass value="0.1" />
+        <inertia ixx="0.0001" ixy="0.0" ixz="0.0" iyy="0.0001" iyz="0.0" izz="0.0001" />
+      </inertial>
       <visual>
         <geometry>
@@ -22,5 +27,15 @@
         <material name="red" />
       </visual>
+      <collision>
+        <geometry>
+          <cylinder radius="0.05" length="0.02" />
+        </geometry>
+      </collision>
     </link>
+    <gazebo reference="${prefix}_link">
+      <material>
+        Gazebo/Red
+      </material>
+    </gazebo>
   </xacro:macro>
   <link name="base_link" />
@@ -38,5 +53,19 @@
       <material name="gray" />
     </visual>
+    <inertial>
+      <origin xyz="0 0 0" rpy="0 0 0" />
+      <mass value="1.0" />
+      <inertia ixx="0.001" ixy="0.0" ixz="0.0" iyy="0.001" iyz="0.0" izz="0.001" />
+    </inertial>
+    <collision>
+      <origin xyz="0 0 0" rpy="0 0 0" />
+      <geometry>
+        <box size="0.24 0.178 0.06" />
+      </geometry>
+    </collision>
   </link>
+  <gazebo reference="body_link">
+    <material>Gazebo/Gray</material>
+  </gazebo>
   <xacro:wheel_macro parent="base_link" prefix="left_wheel" xyz="0 0.1 0.05" />
   <xacro:wheel_macro parent="base_link" prefix="right_wheel" xyz="0 -0.1 0.05" />
@@ -54,4 +83,14 @@
       <color name="gray" />
     </visual>
+    <collision>
+      <origin xyz="0 0 0" rpy="0 0 0" />
+      <geometry>
+        <sphere radius="0.04" />
+      </geometry>
+      <material name="gray" />
+    </collision>
   </link>
+  <gazebo reference="ball_link">
+    <material>Gazebo/Gray</material>
+  </gazebo>
 </robot>

File: catkin_ws/src/vis_lecture/xacro/tire.xacro (robot description, xacro)
@@ -1,8 +1,9 @@
 <robot xmlns:xacro="http://ros.org/wiki/xacro">
   <xacro:macro name="make_tire" params="suffix parent xyz rpy radius length">
-    <joint name="${suffix}_joint" type="fixed">
+    <joint name="${suffix}_joint" type="continuous">
       <parent link="${parent}" />
       <child link="${suffix}_link" />
       <origin xyz="${xyz}" rpy="${rpy}" />
+      <axis xyz="0 0 1" />
     </joint>
     <link name="${suffix}_link">

Commit message: add original vehicle

File: catkin_ws/src/vis_lecture/xacro/body.xacro (robot description, xacro)
@@ -1,3 +1,4 @@
-<robot name="test_robot" xmlns:xacro="http://ros.org/wiki/xacro">
+<robot name="test_robot"
+  xmlns:xacro="http://ros.org/wiki/xacro">
   <xacro:property name="gcolor" value="0 1 0 2.0" />
   <xacro:property name="tire_width" value="0.03" />
@@ -13,6 +14,6 @@
   </link>
   <joint name="body_joint" type="fixed">
-    <parent link="base_link"/>
-    <child  link="body_link"/>
+    <parent link="base_link" />
+    <child link="body_link" />
     <origin xyz="0 0 ${tire_height}" rpy="0 0 0" />
   </joint>
@@ -20,13 +21,29 @@
     <visual>
       <geometry>
-        <box size="0.4 0.4 0.01"/>
+        <box size="0.4 0.4 0.01" />
       </geometry>
-      <origin xyz="0 0 0" rpy="0 0 0"/>
+      <origin xyz="0 0 0" rpy="0 0 0" />
       <material name="green" />
     </visual>
+    <inertial>
+      <origin xyz="0 0 0" rpy="0 0 0" />
+      <mass value="1.0" />
+      <inertia ixx="0.001" ixy="0.0" ixz="0.0" iyy="0.001" iyz="0.0" izz="0.001" />
+    </inertial>
+    <collision>
+      <origin xyz="0 0 0" rpy="0 0 0" />
+      <geometry>
+        <box size="0.4 0.4 0.01" />
+      </geometry>
+    </collision>
   </link>
-  <xacro:make_tire suffix="tire0" parent="body_link" xyz="${body_width/2} ${body_height/2+tire_width/2} 0" rpy="0 1.57 -1.57" radius="${tire_height}" length="${tire_width}"/>
-  <xacro:make_tire suffix="tire1" parent="body_link" xyz="${-(body_width/2)} ${body_height/2+tire_width/2} 0" rpy="0 1.57 -1.57" radius="${tire_height}" length="${tire_width}"/>
-  <xacro:make_tire suffix="tire2" parent="body_link" xyz="${body_width/2} ${-(body_height/2+tire_width/2)} 0" rpy="0 1.57 1.57" radius="${tire_height}" length="${tire_width}"/>
-  <xacro:make_tire suffix="tire3" parent="body_link" xyz="${-(body_width/2)} ${-(body_height/2+tire_width/2)} 0" rpy="0 1.57 1.57" radius="${tire_height}" length="${tire_width}"/>
+  <gazebo reference="body_link">
+    <material>
+      Gazebo/Green
+    </material>
+  </gazebo>
+  <xacro:make_tire suffix="tire0" parent="body_link" xyz="${body_width/2} ${body_height/2+tire_width/2} 0" rpy="0 1.57 -1.57" radius="${tire_height}" length="${tire_width}" />
+  <xacro:make_tire suffix="tire1" parent="body_link" xyz="${-(body_width/2)} ${body_height/2+tire_width/2} 0" rpy="0 1.57 -1.57" radius="${tire_height}" length="${tire_width}" />
+  <xacro:make_tire suffix="tire2" parent="body_link" xyz="${body_width/2} ${-(body_height/2+tire_width/2)} 0" rpy="0 1.57 1.57" radius="${tire_height}" length="${tire_width}" />
+  <xacro:make_tire suffix="tire3" parent="body_link" xyz="${-(body_width/2)} ${-(body_height/2+tire_width/2)} 0" rpy="0 1.57 1.57" radius="${tire_height}" length="${tire_width}" />
 </robot>

File: catkin_ws/src/vis_lecture/xacro/tire.xacro (robot description, xacro)
@@ -17,5 +17,20 @@
         <origin xyz="0 0 0" rpy="0 0 0" />
       </visual>
+      <inertial>
+        <mass value="0.1" />
+        <origin xyz="0 0 0" rpy="0 0 0" />
+        <inertia ixx="0.0001" ixy="0.0" ixz="0.0" iyy="0.0001" iyz="0.0" izz="0.0001" />
+      </inertial>
+      <collision>
+        <geometry>
+          <cylinder radius="${radius}" length="${length}" />
+        </geometry>
+      </collision>
     </link>
+    <gazebo reference="${suffix}_link">
+      <material>
+        Gazebo/Gray
+      </material>
+    </gazebo>
   </xacro:macro>
 </robot>
